File: Hardware/SmartWatch/SmartWatch.sch (EAGLE design)
At the start: 1 part

Commit message: adding things to library
Parts:
- added U2: (no value), SmartWatch:NRF51822_MODULE_MDBT40
- U1: value (none) -> STM32L476; device SmartWatch:NRF51822_MODULE_MDBT40 -> SmartWatch:STM32L476
Changed lines of the file:
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@@
 <setting verticaltext="up"/>
 </settings>
-<grid distance="0.1" unitdist="inch" unit="inch" style="lines" multiple="1" display="no" altdistance="0.01" altunitdist="inch" altunit="inch"/>
+<grid distance="0.05" unitdist="inch" unit="inch" style="lines" multiple="1" display="yes" altdistance="0.005" altunitdist="inch" altunit="inch"/>
 <layers>
 <layer number="1" name="Top" color="4" fill="1" visible="no" active="no"/>
@@
 </classes>
 <parts>
-<part name="U1" library="SmartWatch" deviceset="NRF51822_MODULE_MDBT40" device=""/>
+<part name="U2" library="SmartWatch" deviceset="NRF51822_MODULE_MDBT40" device=""/>
+<part name="U1" library="SmartWatch" deviceset="STM32L476" device=""/>
 </parts>
 <sheets>
@@
 </plain>
 <instances>
-<instance part="U1" gate="G$1" x="78.74" y="68.58"/>
+<instance part="U2" gate="G$1" x="78.74" y="68.58"/>
+<instance part="U1" gate="PORTA" x="27.94" y="-20.32"/>
+<instance part="U1" gate="PORTB" x="57.15" y="-20.32"/>
+<instance part="U1" gate="PORTC" x="88.9" y="-20.32"/>
+<instance part="U1" gate="G$4" x="57.15" y="-67.31"/>
 </instances>
 <busses>

Commit message: Continued work on schematic and libraries
Parts:
- added C1, C14, C3: 1uF, microbuilder:CAP_CERAMIC0603MINI
- added C10: 1.0uF, microbuilder:CAP_CERAMIC0603MINI
- added C11, C4, C5, C8: 0.1uF, microbuilder:CAP_CERAMIC0603MINI
- added C12: 47uF, resistor:C-EUC1206
- added C2, C6: 10uF/16V, microbuilder:CAP_CERAMIC0603MINI
- added C7, C9: 10uF, microbuilder:CAP_CERAMIC0603MINI
- added D1, D3: 1N4148, microbuilder:DIODESOD-323
- added D2: BAT54T1G, microbuilder:DIODESOD-123
- added L1: 10uH, microbuilder:INDUCTOR
- added R1, R10, R11, R12, R2: 10k, resistor:R-US_R0603
- added R3, R8: 4.7k, resistor:R-US_R0603
- added R4: 600K, resistor:R-US_R0603
- added R5: 50, resistor:R-US_R0603
- added R6: 100K, resistor:R-US_R0603
- added R7, R9: 10K, resistor:R-US_R0603
- added U$27: LTC3557, SmartWatch:LTC3557
- added U$5: BNO055, SmartWatch:BNO055
- added U3: UG-2828GDEDF11, microbuilder:DISP_OLED_UG-2828GDEDF11TOP
- added U4: FAN5331SX, microbuilder:FAN5331
- added U5: APDS-9960, SparkFun-Sensors:APDS-9960
Connections:
- new net +3V3: C1.2, R1.2, U2.AVDD, U2.VDD
- new net 13V: C2.2, C8.1, D2.C, R6.2, U3.VCC
- new net 3.3V: C10.2, C11.2, C12.1, C3.2, C5.2, C7.1, C9.2, L1.1, R3.2, R8.2, R9.2, U$5.NBOOT, U$5.VDD, U$5.VDDIO, U3.VCI, U3.VDDIO, U4.SHDN, U4.VIN, U5.LEDA, U5.VDD
- new net BT_CS: R1.1, U2.P0.24
- new net BT_IRQ: U2.P0.25
- new net BT_MISO: U2.P0.22
- new net BT_MOSI: U2.P0.23
- new net BT_SCK: U2.P0.21
- new net GND: C1.1, C10.1, C11.1, C12.2, C14.1, C2.1, C3.1, C4.1, C5.1, C6.2, C7.2, C9.1, D3.C, R10.2, R11.1, R12.1, R2.1, R4.1, R7.1, U$5.GND10, U$5.GND15, U$5.GND16, U$5.GND18, U$5.GND2, U$5.GND25, U2.GND@1, U2.GND@2, U2.GND@3, U2.GND@4, U2.GND@5, U2.P0.30, U3.BS1, U3.NC(GND)@1, U3.NC(GND)@2, U3.VSS, U4.GND, U5.GND
- new net G_INT: R9.1, U5.INT
- new net IMU_INT: U$5.INT
- new net IMU_NRESET: U$5.NRESET
- new net MOSI/DATA1: U3.D1/SDIN
- new net N$1: R4.2, U3.IREF
- new net N$11: D1.C, D3.A
- new net N$13: R12.2, U$5.PS1
- new net N$14: R11.2, U$5.PS0
- new net N$2: C14.2, U3.VDD
- new net N$3: R10.1, U$5.I2C_ADDR
- new net N$4: C4.2, U$5.CAP
- new net N$5: D2.A, L1.2, U4.SW
- new net N$6: R5.2, U3.VSL
- new net N$7: D1.A, R5.1
- new net N$8: C8.2, R6.1, R7.2, U4.FB
- new net N$9: U5.LDR, U5.LEDK
- new net OLED_BS0: R2.2, U3.BS0
- new net OLED_CS: U3.CS#
- new net OLED_DC: U3.D/C#
- new net OLED_RES: U3.RES#
- new net SCK/DATA0: U3.D0/SCK
- new net SCL: R3.1, U$5.SCL/RX, U5.SCL
- new net SDA: R8.1, U$5.SDA/TX, U5.SDA
- new net VCOMH1: C6.1, U3.VCOMH
Other:
- note added: "13V Boost"
- note added: "Bluetooth Module"
- note added: "Gesture Sensor"
- note added: "IMU"
- note added: "OLED Display"
- note added: "VOUT = 1.23V * (1 + R6/R7)"
- note added: "VOUT = 13.53V"

Commit message: renamed part
Parts:
- renumbered U$27 to U6
Changed lines of the file:
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@@
 <part name="C12" library="resistor" deviceset="C-EU" device="C1206" value="47uF"/>
 <part name="C1" library="microbuilder" deviceset="CAP_CERAMIC" device="0603MINI" value="1uF"/>
-<part name="U$27" library="SmartWatch" deviceset="LTC3557" device=""/>
+<part name="U6" library="SmartWatch" deviceset="LTC3557" device=""/>
 </parts>
 <sheets>
@@
 <instance part="C12" gate="G$1" x="241.3" y="5.08"/>
 <instance part="C1" gate="G$1" x="13.97" y="69.85" rot="R180"/>
-<instance part="U$27" gate="G$1" x="198.12" y="-48.26"/>
+<instance part="U6" gate="G$1" x="198.12" y="-48.26"/>
 </instances>
 <busses>

Commit message: Updated schematic
Parts:
- added JP1: (no value), SparkFun-Connectors:USB_MICROB_PLUGCONN-11752
- added RN1: (no value), MicroBoard:2R-NEXBV4V
Connections:
- new net D+: RN1A.2
- new net D-: RN1B.2
- new net N$10: JP1.D+, RN1A.1
- new net N$15: JP1.D-, RN1B.1
Changed lines of the file:
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@@
 <part name="C1" library="microbuilder" deviceset="CAP_CERAMIC" device="0603MINI" value="1uF"/>
 <part name="U6" library="SmartWatch" deviceset="LTC3557" device=""/>
+<part name="JP1" library="SparkFun-Connectors" deviceset="USB_MICROB_PLUG" device="CONN-11752"/>
+<part name="RN1" library="MicroBoard" deviceset="2R-N" device="EXBV4V"/>
 </parts>
 <sheets>
@@
 <instance part="C1" gate="G$1" x="13.97" y="69.85" rot="R180"/>
 <instance part="U6" gate="G$1" x="198.12" y="-48.26"/>
+<instance part="JP1" gate="G$1" x="158.75" y="1.27" rot="R180"/>
+<instance part="RN1" gate="A" x="187.96" y="2.54"/>
+<instance part="RN1" gate="B" x="187.96" y="-2.54"/>
 </instances>
 <busses>
@@
 </segment>
 </net>
+<net name="N$10" class="0">
+<segment>
+<pinref part="JP1" gate="G$1" pin="D+"/>
+<wire x1="166.37" y1="1.27" x2="180.34" y2="1.27" width="0.1524" layer="91"/>
+<wire x1="180.34" y1="1.27" x2="180.34" y2="2.54" width="0.1524" layer="91"/>
+<pinref part="RN1" gate="A" pin="1"/>
+<wire x1="180.34" y1="2.54" x2="182.88" y2="2.54" width="0.1524" layer="91"/>
+</segment>
+</net>
+<net name="N$15" class="0">
+<segment>
+<pinref part="JP1" gate="G$1" pin="D-"/>
+<wire x1="166.37" y1="-1.27" x2="177.8" y2="-1.27" width="0.1524" layer="91"/>
+<wire x1="177.8" y1="-1.27" x2="177.8" y2="-2.54" width="0.1524" layer="91"/>
+<pinref part="RN1" gate="B" pin="1"/>
+<wire x1="177.8" y1="-2.54" x2="182.88" y2="-2.54" width="0.1524" layer="91"/>
+</segment>
+</net>
+<net name="D+" class="0">
+<segment>
+<pinref part="RN1" gate="A" pin="2"/>
+<wire x1="193.04" y1="2.54" x2="195.58" y2="2.54" width="0.1524" layer="91"/>
+<label x="195.58" y="2.54" size="1.27" layer="95" xref="yes"/>
+</segment>
+</net>
+<net name="D-" class="0">
+<segment>
+<pinref part="RN1" gate="B" pin="2"/>
+<wire x1="193.04" y1="-2.54" x2="195.58" y2="-2.54" width="0.1524" layer="91"/>
+<label x="195.58" y="-2.54" size="1.27" layer="95" xref="yes"/>
+</segment>
+</net>

Commit message: added to schematic more
Parts:
- added U$16, U$28, U$29, U$30, U$31, U$32: PTS840-GM, SmartWatch:PTS840-GM
- U3: device microbuilder:DISP_OLED_UG-2828GDEDF11TOP -> SmartWatch:DISP_OLED_UG-2828GDEDF11BOTTOM
- U4: device microbuilder:FAN5331 -> SmartWatch:FAN5331
Changed lines of the file:
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@@
 <part name="R5" library="resistor" deviceset="R-US_" device="R0603" value="50"/>
 <part name="D1" library="microbuilder" deviceset="DIODE" device="SOD-323" value="1N4148"/>
-<part name="U$8" library="microbuilder" deviceset="13V" device=""/>
+<part name="U$8" library="supply1" deviceset="+12V" device="" value="+13V"/>
 <part name="U$7" library="microbuilder" deviceset="3.3V" device=""/>
 <part name="U$1" library="microbuilder" deviceset="3.3V" device=""/>
-<part name="U3" library="microbuilder" deviceset="DISP_OLED_UG-2828GDEDF11" device="TOP" value="UG-2828GDEDF11"/>
+<part name="U3" library="SmartWatch" deviceset="DISP_OLED_UG-2828GDEDF11" device="BOTTOM" value="UG-2828GDEDF11"/>
 <part name="C6" library="microbuilder" deviceset="CAP_CERAMIC" device="0603MINI" value="10uF/16V"/>
 <part name="D3" library="microbuilder" deviceset="DIODE" device="SOD-323" value="1N4148"/>
 <part name="U$3" library="microbuilder" deviceset="GND" device=""/>
 <part name="R2" library="resistor" deviceset="R-US_" device="R0603" value="10k"/>
-<part name="U4" library="microbuilder" deviceset="FAN5331" device="" value="FAN5331SX"/>
+<part name="U4" library="SmartWatch" deviceset="FAN5331" device="" value="FAN5331SX"/>
 <part name="C7" library="microbuilder" deviceset="CAP_CERAMIC" device="0603MINI" value="10uF"/>
 <part name="L1" library="microbuilder" deviceset="INDUCTOR" device="" value="10uH"/>
@@
 <part name="U$13" library="microbuilder" deviceset="GND" device=""/>
 <part name="C8" library="microbuilder" deviceset="CAP_CERAMIC" device="0603MINI" value="0.1uF"/>
-<part name="U$16" library="microbuilder" deviceset="13V" device=""/>
 <part name="U$15" library="microbuilder" deviceset="3.3V" device=""/>
 <part name="U$2" library="microbuilder" deviceset="GND" device=""/>
@@
 <part name="JP1" library="SparkFun-Connectors" deviceset="USB_MICROB_PLUG" device="CONN-11752"/>
 <part name="RN1" library="MicroBoard" deviceset="2R-N" device="EXBV4V"/>
+<part name="U$27" library="supply1" deviceset="+12V" device="" value="+13V"/>
+<part name="U$16" library="SmartWatch" deviceset="PTS840-GM" device=""/>
+<part name="U$28" library="SmartWatch" deviceset="PTS840-GM" device=""/>
+<part name="U$29" library="SmartWatch" deviceset="PTS840-GM" device=""/>
+<part name="U$30" library="SmartWatch" deviceset="PTS840-GM" device=""/>
+<part name="U$31" library="SmartWatch" deviceset="PTS840-GM" device=""/>
+<part name="U$32" library="SmartWatch" deviceset="PTS840-GM" device=""/>
 </parts>
 <sheets>
@@
 <instance part="R5" gate="G$1" x="173.99" y="96.52"/>
 <instance part="D1" gate="G$1" x="165.1" y="93.98" rot="R270"/>
-<instance part="U$8" gate="G$1" x="175.26" y="114.3"/>
+<instance part="U$8" gate="1" x="175.26" y="114.3"/>
 <instance part="U$7" gate="G$1" x="171.45" y="33.02" rot="R180"/>
 <instance part="U$1" gate="G$1" x="166.37" y="114.3"/>
@@
 <instance part="U$13" gate="G$1" x="275.59" y="54.61"/>
 <instance part="C8" gate="G$1" x="298.45" y="80.01"/>
-<instance part="U$16" gate="G$1" x="298.45" y="92.71"/>
 <instance part="U$15" gate="G$1" x="234.95" y="92.71"/>
 <instance part="U$2" gate="G$1" x="134.62" y="78.74"/>
@@
 <instance part="RN1" gate="A" x="187.96" y="2.54"/>
 <instance part="RN1" gate="B" x="187.96" y="-2.54"/>
+<instance part="U$27" gate="1" x="298.45" y="92.71"/>
+<instance part="U$16" gate="G$1" x="298.45" y="-15.24"/>
+<instance part="U$28" gate="G$1" x="298.45" y="-22.86"/>
+<instance part="U$29" gate="G$1" x="298.45" y="-29.21"/>
+<instance part="U$30" gate="G$1" x="298.45" y="-38.1"/>
+<instance part="U$31" gate="G$1" x="298.45" y="-44.45"/>
+<instance part="U$32" gate="G$1" x="298.45" y="-49.53"/>
 </instances>
 <busses>
@@
 <junction x="175.26" y="104.14"/>
 <pinref part="C2" gate="G$1" pin="2"/>
-<pinref part="U$8" gate="G$1" pin="13V"/>
+<pinref part="U$8" gate="1" pin="+12V"/>
 <pinref part="U3" gate="G$1" pin="VCC"/>
 </segment>
@@
 <wire x1="283.21" y1="90.17" x2="290.83" y2="90.17" width="0.1524" layer="91"/>
 <junction x="290.83" y="90.17"/>
-<junction x="298.45" y="90.17"/>
 <pinref part="C8" gate="G$1" pin="1"/>
 <pinref part="R6" gate="G$1" pin="2"/>
 <pinref part="D2" gate="G$1" pin="C"/>
-<pinref part="U$16" gate="G$1" pin="13V"/>
-</segment>
-</net>
+<pinref part="U$27" gate="1" pin="+12V"/>
+<junction x="298.45" y="90.17"/>
+</segment>
+</net>
